Commit message: updated images

File: src/testbot_description/urdf/my_robot.urdf.xacro (robot description, xacro)
@@ -22,5 +22,5 @@
         <collision>
             <geometry>
-                <box size="0.8 0.7 0.1" />
+                <box size="${width_base} ${height_base} ${depth_base}" />
             </geometry>
         </collision>
