Commit message: added intel realsense camera

File: src/testbot_description/urdf/gazebo.xacro (robot description, xacro)
@@ -32,3 +32,146 @@
     <xacro:wheel_trans name ="front_right"/>
     <xacro:wheel_trans name ="front_left"/>
+    <!-- Realsense D435i -->
+    <gazebo reference="camera_color_frame">
+    <sensor name="color" type="camera">
+        <pose frame="">0 0 0 0 0 0</pose>
+        <camera name="__default__">
+        <horizontal_fov>1.5009831567151233</horizontal_fov>
+        <image>
+            <width>640</width>
+            <height>480</height>
+            <format>RGB_INT8</format>
+        </image>
+        <clip>
+            <near>0.1</near>
+            <far>100</far>
+        </clip>
+        <noise>
+            <type>gaussian</type>
+            <mean>0.0</mean>
+            <stddev>0.007</stddev>
+        </noise>
+        </camera>
+        <always_on>1</always_on>
+        <update_rate>30</update_rate>
+        <visualize>0</visualize>
+    </sensor>
+    </gazebo>
+    <gazebo reference="camera_infra1_frame">
+    <sensor name="ired1" type="camera">
+        <pose frame="">0 0 0 0 0 0</pose>
+        <camera name="__default__">
+        <horizontal_fov>1.5009831567151233</horizontal_fov>
+        <image>
+            <width>640</width>
+            <height>480</height>
+            <format>L_INT8</format>
+        </image>
+        <clip>
+            <near>0.1</near>
+            <far>100</far>
+        </clip>
+        <noise>
+            <type>gaussian</type>
+            <mean>0.0</mean>
+            <stddev>0.007</stddev>
+        </noise>
+        </camera>
+        <always_on>1</always_on>
+        <update_rate>30</update_rate>
+        <visualize>0</visualize>
+    </sensor>
+    </gazebo>
+    <gazebo reference="camera_infra2_frame">
+    <sensor name="ired2" type="camera">
+        <pose frame="">0 0 0 0 0 0</pose>
+        <camera name="__default__">
+        <horizontal_fov>1.5009831567151233</horizontal_fov>
+        <image>
+            <width>640</width>
+            <height>480</height>
+            <format>L_INT8</format>
+        </image>
+        <clip>
+            <near>0.1</near>
+            <far>100</far>
+        </clip>
+        <noise>
+            <type>gaussian</type>
+            <mean>0.0</mean>
+            <stddev>0.007</stddev>
+        </noise>
+        </camera>
+        <always_on>1</always_on>
+        <update_rate>30</update_rate>
+        <visualize>0</visualize>
+    </sensor>
+    </gazebo>
+    <gazebo reference="camera_depth_frame">
+    <sensor name="depth" type="depth">
+        <pose frame="">0 0 0 0 0 0</pose>
+        <camera name="__default__">
+        <horizontal_fov>1.5009831567151233</horizontal_fov>
+        <image>
+            <width>640</width>
+            <height>480</height>
+        </image>
+        <clip>
+            <near>0.1</near>
+            <far>100</far>
+        </clip>
+        <noise>
+            <type>gaussian</type>
+            <mean>0.0</mean>
+            <stddev>0.007</stddev>
+        </noise>
+        </camera>
+        <always_on>1</always_on>
+        <update_rate>30</update_rate>
+        <visualize>0</visualize>
+    </sensor>
+    </gazebo>
+    <gazebo>
+        <plugin name="camera" filename="librealsense_gazebo_plugin.so">
+        <depthUpdateRate>30</depthUpdateRate>
+        <colorUpdateRate>30</colorUpdateRate>
+        <infraredUpdateRate>30</infraredUpdateRate>
+        <depthTopicName>depth/image_raw</depthTopicName>
+        <depthCameraInfoTopicName>depth/camera_info</depthCameraInfoTopicName>
+        <colorTopicName>color/image_raw</colorTopicName>
+        <colorCameraInfoTopicName>color/camera_info</colorCameraInfoTopicName>
+        <infrared1TopicName>infrared/image_raw</infrared1TopicName>
+        <infrared1CameraInfoTopicName>infrared/camera_info</infrared1CameraInfoTopicName>
+        <infrared2TopicName>infrared2/image_raw</infrared2TopicName>
+        <infrared2CameraInfoTopicName>infrared2/camera_info</infrared2CameraInfoTopicName>
+        <colorOpticalframeName>camera_color_optical_frame</colorOpticalframeName>
+        <depthOpticalframeName>camera_depth_optical_frame</depthOpticalframeName>
+        <infrared1OpticalframeName>camera_left_ir_optical_frame</infrared1OpticalframeName>
+        <infrared2OpticalframeName>camera_right_ir_optical_frame</infrared2OpticalframeName>
+        <rangeMinDepth>0.1</rangeMinDepth>
+        <rangeMaxDepth>10</rangeMaxDepth>
+        <pointCloud>1</pointCloud>
+        <pointCloudTopicName>depth/color/points</pointCloudTopicName>
+        <pointCloudCutoff>0.15</pointCloudCutoff>
+        <pointCloudCutoffMax>10</pointCloudCutoffMax>
+        </plugin>
+    </gazebo>
+    <gazebo reference="camera_gyro_frame">
+    <gravity>true</gravity>
+    <sensor name="imu_sensor" type="imu">
+        <always_on>true</always_on>
+        <visualize>false</visualize>
+        <plugin name="imu_plugin" filename="libgazebo_ros_imu_sensor.so">
+        <topicName>camera/imu/data</topicName>
+        <bodyName>camera_gyro_frame</bodyName>
+        <updateRateHZ>50.0</updateRateHZ>
+        <gaussianNoise>0.001</gaussianNoise>
+        <xyzOffset>0 0 0</xyzOffset>
+        <rpyOffset>0 0 0</rpyOffset>
+        <frameName>camera_gyro_frame</frameName>
+        <initialOrientationAsReference>false</initialOrientationAsReference>
+        </plugin>
+        <pose>0 0 0 0 0 0</pose>
+    </sensor>
+    </gazebo>
 </robot>

File: src/testbot_description/urdf/my_robot.urdf.xacro (robot description, xacro)
@@ -3,10 +3,10 @@
     <xacro:property name="constant" value="0.083"/>
     <xacro:property name="mass_base" value="1.0"/>
-    <xacro:property name="width_base" value="0.8"/>
-    <xacro:property name="height_base" value="0.7"/>
+    <xacro:property name="width_base" value="0.6"/>
+    <xacro:property name="height_base" value="0.5"/>
     <xacro:property name="depth_base" value="0.1"/>
-    <xacro:property name="mass_wheel" value="0.5"/>
-    <xacro:property name="height_wheel" value="0.1"/>
-    <xacro:property name="radius_wheel" value="0.16"/>
+    <xacro:property name="mass_wheel" value="0.3"/>
+    <xacro:property name="height_wheel" value="0.07"/>
+    <xacro:property name="radius_wheel" value="0.1"/>
     <!-- Robot Base  -->
     <link name="base_link">
@@ -39,5 +39,5 @@
                 <geometry>
                     <!-- <mesh filename="package://testbot_description/meshes/${type}_tire.stl" scale="0.005 0.005 0.005"/> -->
-                    <cylinder radius="0.16" length="0.1"/>
+                    <cylinder radius="${radius_wheel}" length="${height_wheel}"/>
                 </geometry>
                 <material name="LightGrey">
@@ -48,5 +48,5 @@
                 <geometry>
                     <!-- <mesh filename="package://testbot_description/meshes/${type}_tire.stl" scale="0.005 0.005 0.005"/> -->
-                    <cylinder radius="0.16" length="0.1"/>
+                    <cylinder radius="${radius_wheel}" length="${height_wheel}"/>
                 </geometry>
             </collision>
@@ -65,12 +65,39 @@
             <axis xyz="0 1 0"/> -->
             <origin xyz="${x} ${y} 0" rpy="1.57 0 0"/>
-            <axis xyz="0 0 -1"/>
+            <axis xyz="0 0 1"/>
         </joint>
     </xacro:macro>
-    <!-- Rear Right Wheel (created using macro)-->
-    <xacro:wheel name ="rear_right" x ="0.25" y="0.40" type="right"/>
-    <xacro:wheel name ="rear_left" x ="0.25" y="-0.40" type="left"/>
-    <xacro:wheel name ="front_right" x ="-0.25" y="0.40" type="right"/>
-    <xacro:wheel name ="front_left" x ="-0.25" y="-0.40" type="left"/>
+    <!-- Wheels (created using macro)-->
+    <xacro:wheel name ="rear_right" x ="0.30" y="0.285" type="right"/>
+    <xacro:wheel name ="rear_left" x ="0.30" y="-0.285" type="left"/>
+    <xacro:wheel name ="front_right" x ="-0.30" y="0.285" type="right"/>
+    <xacro:wheel name ="front_left" x ="-0.30" y="-0.285" type="left"/>
+    <link name="realsense_camera_link">
+        <visual>
+            <geometry>
+                <box size="0.09 0.025 0.025" />
+            </geometry>
+            <material name="LightGrey">
+                <color rgba="0.7 0.7 0.7 1.0"/>
+            </material>
+        </visual>
+        <collision>
+            <geometry>
+                <box size="0.09 0.025 0.025" />
+            </geometry>
+        </collision>
+        <inertial>
+            <mass value="0.05"/>
+            <origin xyz="0.0 0.0 0.0" rpy="0.0 0.0 0.0"/>
+            <inertia ixx="0.001" ixy="0.0" ixz="0.0" iyy="0.001" iyz="0.0" izz="0.001"/>
+        </inertial>
+    </link>
+    <joint name="realsense_camera_joint" type="fixed">
+        <parent link="base_link"/>
+        <child link="realsense_camera_link"/>
+        <origin xyz="-0.2875 0 0.0625" rpy="0 0 -1.57"/>
+        <axis xyz="0 0 0"/>
+    </joint>
     <xacro:include filename="gazebo.xacro"/>
+    <xacro:include filename="testbot_d435i.xacro"/>
 </robot>

Commit message: fixed bugs

File: src/testbot_description/urdf/gazebo.xacro (robot description, xacro)
@@ -6,9 +6,7 @@
     <!-- Gazebo plugin for ROS Control -->
     <gazebo>
-        <plugin name="gazebo_ros_control" filename="libgazebo_ros_control.so">
-            <robotNamespace>/</robotNamespace>
-        </plugin>
-    </gazebo>
-    <xacro:macro name="wheel_trans" params="name">
+        <plugin name="gazebo_ros_control" filename="libgazebo_ros_control.so"/>
+    </gazebo>
+    <!-- <xacro:macro name="wheel_trans" params="name mu1 mu2">
         <transmission name="wheel_${name}_trans">
             <type>transmission_interface/SimpleTransmission</type>
@@ -21,16 +19,181 @@
         </transmission>
         <gazebo reference="wheel_${name}_link">
-            <mu1 value="200.0"/>
-            <mu2 value="100.0"/>
+            <mu1 value="${mu1}"/>
+            <mu2 value="${mu2}"/>
             <kp value="10000000.0" />
             <kd value="1.0" />
             <material>Gazebo/DarkGrey</material>
         </gazebo>
-    </xacro:macro>
-    <xacro:wheel_trans name ="rear_right"/>
-    <xacro:wheel_trans name ="rear_left"/>
-    <xacro:wheel_trans name ="front_right"/>
-    <xacro:wheel_trans name ="front_left"/>
-    <!-- Realsense D435i -->
+    </xacro:macro> -->
+<gazebo reference="wheel_front_right_link">
+  <material>Gazebo/DarkGrey</material>
+  <mu1>0.5</mu1>
+  <mu2>0.5</mu2>
+  <selfCollide>true</selfCollide>
+</gazebo>
+<gazebo reference="wheel_front_left_link">
+  <material>Gazebo/DarkGrey</material>
+  <mu1>0.5</mu1>
+  <mu2>0.5</mu2>
+  <selfCollide>true</selfCollide>
+</gazebo>
+<gazebo reference="wheel_rear_right_link">
+  <material>Gazebo/DarkGrey</material>
+  <mu1>0.001</mu1>
+  <mu2>0.001</mu2>
+  <selfCollide>true</selfCollide>
+</gazebo>
+<gazebo reference="wheel_rear_left_link">
+  <material>Gazebo/DarkGrey</material>
+  <mu1>0.001</mu1>
+  <mu2>0.001</mu2>
+  <selfCollide>true</selfCollide>
+</gazebo>
+    <!-- <xacro:wheel_trans name ="rear_right" mu1 ="0.01" mu2 = "0.01"/>
+    <xacro:wheel_trans name ="rear_left" mu1 ="0.01" mu2 = "0.01"/> -->
+    <!-- <xacro:wheel_trans name ="front_right" mu1 ="200" mu2 = "100"/>
+    <xacro:wheel_trans name ="front_left" mu1 ="200" mu2 = "100"/> -->
+    <joint name="camera_optical_joint" type="fixed">
+        <origin xyz="0 0 0" rpy="-1.571 0 -1.571" />
+        <parent link="camera_link" />
+        <child link="camera_link_optical" />
+    </joint>
+    <link name="camera_link_optical"></link>
+    <xacro:property name="link_name" value="camera_link"/>
+    <xacro:property name="camera_name" value="camera"/>
+    <xacro:property name="frame_name" value="camera_link_optical"/>
+    <gazebo reference="${link_name}">
+        <sensor name="my_camera" type="depth">
+            <update_rate>20</update_rate>
+            <camera>
+            <horizontal_fov>1.047198</horizontal_fov>
+            <image>
+                <width>640</width>
+                <height>480</height>
+                <format>R8G8B8</format>
+            </image>
+            <clip>
+                <near>0.05</near>
+                <far>3</far>
+            </clip>
+            </camera>
+            <plugin name="${camera_name}_controller" filename="libgazebo_ros_openni_kinect.so">
+            <baseline>0.2</baseline>
+            <alwaysOn>true</alwaysOn>
+            <updateRate>1.0</updateRate>
+            <cameraName>${camera_name}_ir</cameraName>
+            <imageTopicName>/${camera_name}/color/image_raw</imageTopicName>
+            <cameraInfoTopicName>/${camera_name}/color/camera_info</cameraInfoTopicName>
+            <depthImageTopicName>/${camera_name}/depth/image_raw</depthImageTopicName>
+            <depthImageInfoTopicName>/${camera_name}/depth/camera_info</depthImageInfoTopicName>
+            <pointCloudTopicName>/${camera_name}/depth/points</pointCloudTopicName>
+            <frameName>${frame_name}</frameName>
+            <pointCloudCutoff>0.5</pointCloudCutoff>
+            <pointCloudCutoffMax>3.0</pointCloudCutoffMax>
+            <distortionK1>0.00000001</distortionK1>
+            <distortionK2>0.00000001</distortionK2>
+            <distortionK3>0.00000001</distortionK3>
+            <distortionT1>0.00000001</distortionT1>
+            <distortionT2>0.00000001</distortionT2>
+            <CxPrime>0</CxPrime>
+            <Cx>0</Cx>
+            <Cy>0</Cy>
+            <focalLength>0</focalLength>
+            <hackBaseline>0</hackBaseline>
+            </plugin>
+        </sensor>
+    </gazebo>
+    <gazebo>
+        <plugin name="turtlebot3_waffle_controller" filename="libgazebo_ros_diff_drive.so">
+        <commandTopic>cmd_vel</commandTopic>
+        <odometryTopic>odom</odometryTopic>
+        <odometryFrame>odom</odometryFrame>
+        <odometrySource>world</odometrySource>
+        <publishOdomTF>true</publishOdomTF>
+        <robotBaseFrame>base_link</robotBaseFrame>
+        <publishWheelTF>false</publishWheelTF>
+        <publishTf>true</publishTf>
+        <publishWheelJointState>true</publishWheelJointState>
+        <legacyMode>false</legacyMode>
+        <updateRate>30</updateRate>
+        <leftJoint>wheel_front_left_joint</leftJoint>
+        <rightJoint>wheel_front_right_joint</rightJoint>
+        <leftJoint>wheel_rear_left_joint</leftJoint>
+        <rightJoint>wheel_rear_right_joint</rightJoint>
+        <wheelSeparation>0.4</wheelSeparation>
+        <wheelDiameter>0.2</wheelDiameter>
+        <wheelAcceleration>1</wheelAcceleration>
+        <wheelTorque>100</wheelTorque>
+        <rosDebugLevel>na</rosDebugLevel>
+        </plugin>
+  </gazebo>
+  <!-- <gazebo>
+    <plugin name="imu_plugin" filename="libgazebo_ros_imu.so">
+      <alwaysOn>true</alwaysOn>
+      <bodyName>imu_link</bodyName>
+      <frameName>imu_link</frameName>
+      <topicName>imu</topicName>
+      <serviceName>imu_service</serviceName>
+      <gaussianNoise>0.0</gaussianNoise>
+      <updateRate>0</updateRate>
+      <imu>
+        <noise>
+          <type>gaussian</type>
+          <rate>
+            <mean>0.0</mean>
+            <stddev>2e-4</stddev>
+            <bias_mean>0.0000075</bias_mean>
+            <bias_stddev>0.0000008</bias_stddev>
+          </rate>
+          <accel>
+            <mean>0.0</mean>
+            <stddev>1.7e-2</stddev>
+            <bias_mean>0.1</bias_mean>
+            <bias_stddev>0.001</bias_stddev>
+          </accel>
+        </noise>
+      </imu>
+    </plugin>
+  </gazebo> -->
+  <!-- <gazebo reference="wheel_rear_left_link">
+    <mu1>0.1</mu1>
+    <mu2>0.1</mu2>
+    <kp>500000.0</kp>
+    <kd>10.0</kd>
+    <minDepth>0.001</minDepth>
+    <maxVel>0.1</maxVel>
+    <fdir1>1 0 0</fdir1>
+    <material>Gazebo/FlatBlack</material>
+  </gazebo>
+  <gazebo reference="wheel_rear_right_link">
+    <mu1>0.1</mu1>
+    <mu2>0.1</mu2>
+    <kp>500000.0</kp>
+    <kd>10.0</kd>
+    <minDepth>0.001</minDepth>
+    <maxVel>0.1</maxVel>
+    <fdir1>1 0 0</fdir1>
+    <material>Gazebo/FlatBlack</material>
+  </gazebo>
+  <gazebo reference="wheel_front_right_link">
+    <mu1>0</mu1>
+    <mu2>0</mu2>
+    <kp>1000000.0</kp>
+    <kd>100.0</kd>
+    <minDepth>0.001</minDepth>
+    <maxVel>1.0</maxVel>
+    <material>Gazebo/FlatBlack</material>
+  </gazebo>
+  <gazebo reference="wheel_front_left_link">
+    <mu1>0</mu1>
+    <mu2>0</mu2>
+    <kp>1000000.0</kp>
+    <kd>100.0</kd>
+    <minDepth>0.001</minDepth>
+    <maxVel>1.0</maxVel>
+    <material>Gazebo/FlatBlack</material>
+  </gazebo>
+ -->
+    <!-- Realsense D435i
     <gazebo reference="camera_color_frame">
     <sensor name="color" type="camera">
@@ -174,4 +337,4 @@
         <pose>0 0 0 0 0 0</pose>
     </sensor>
-    </gazebo>
+    </gazebo> -->
 </robot>

File: src/testbot_description/urdf/my_robot.urdf.xacro (robot description, xacro)
@@ -3,10 +3,10 @@
     <xacro:property name="constant" value="0.083"/>
     <xacro:property name="mass_base" value="1.0"/>
-    <xacro:property name="width_base" value="0.6"/>
-    <xacro:property name="height_base" value="0.5"/>
+    <xacro:property name="width_base" value="0.4"/>
+    <xacro:property name="height_base" value="0.3"/>
     <xacro:property name="depth_base" value="0.1"/>
     <xacro:property name="mass_wheel" value="0.3"/>
-    <xacro:property name="height_wheel" value="0.07"/>
-    <xacro:property name="radius_wheel" value="0.1"/>
+    <xacro:property name="height_wheel" value="0.05"/>
+    <xacro:property name="radius_wheel" value="0.08"/>
     <!-- Robot Base  -->
     <link name="base_link">
@@ -27,5 +27,5 @@
         <inertial>
             <origin xyz="0.0 0.0 0.0" rpy="0.0 0.0 0.0"/>
-            <mass value="1.0"/>
+            <mass value="${mass_base}"/>
             <inertia ixx="${constant * mass_base * (depth_base*depth_base + height_base*height_base)}" ixy="0.0" ixz="0.0"
                      iyy="${constant * mass_base * (depth_base*depth_base + width_base*width_base)}" iyz="0.0"
@@ -34,9 +34,9 @@
     </link>
     <!-- Macro for creating wheel -->
-    <xacro:macro name="wheel" params="name x y type">
+    <xacro:macro name="wheel" params="name x y type joint_type">
         <link name="wheel_${name}_link">
             <visual>
                 <geometry>
-                    <!-- <mesh filename="package://testbot_description/meshes/${type}_tire.stl" scale="0.005 0.005 0.005"/> -->
+                    <!-- <mesh filename="package://testbot_description/meshes/${type}_tire.stl" scale="0.003 0.003 0.003"/> -->
                     <cylinder radius="${radius_wheel}" length="${height_wheel}"/>
                 </geometry>
@@ -49,15 +49,16 @@
                     <!-- <mesh filename="package://testbot_description/meshes/${type}_tire.stl" scale="0.005 0.005 0.005"/> -->
                     <cylinder radius="${radius_wheel}" length="${height_wheel}"/>
+                    <!-- <origin xyz="0.0 0.0 0.0" rpy="0.0 1.57 0.0"/> -->
                 </geometry>
             </collision>
             <inertial>
-                <mass value="0.5"/>
+                <mass value="${mass_wheel}"/>
                 <origin xyz="0.0 0.0 0.0" rpy="0.0 0.0 0.0"/>
                 <inertia ixx="${constant * mass_wheel * (3 * radius_wheel * radius_wheel + height_wheel * height_wheel)}" ixy="0.0" ixz="0.0"
-                iyy="${constant * mass_wheel * (3 * radius_wheel * radius_wheel + height_wheel * height_wheel)}" iyz="0.0"
-                izz="${0.5 * mass_wheel * radius_wheel * radius_wheel}"/>
+                         iyy="${constant * mass_wheel * (3 * radius_wheel * radius_wheel + height_wheel * height_wheel)}" iyz="0.0"
+                         izz="${0.5 * mass_wheel * radius_wheel * radius_wheel}"/>
             </inertial>
         </link>
-        <joint name="wheel_${name}_joint" type="continuous">
+        <joint name="wheel_${name}_joint" type="${joint_type}">
             <parent link="base_link"/>
             <child link="wheel_${name}_link"/>
@@ -69,12 +70,18 @@
     </xacro:macro>
     <!-- Wheels (created using macro)-->
-    <xacro:wheel name ="rear_right" x ="0.30" y="0.285" type="right"/>
-    <xacro:wheel name ="rear_left" x ="0.30" y="-0.285" type="left"/>
-    <xacro:wheel name ="front_right" x ="-0.30" y="0.285" type="right"/>
-    <xacro:wheel name ="front_left" x ="-0.30" y="-0.285" type="left"/>
-    <link name="realsense_camera_link">
+    <xacro:wheel name ="rear_right" x ="${width_base/2}" y="${height_base/2 + height_wheel/2}" type="right" joint_type="fixed"/>
+    <xacro:wheel name ="rear_left" x ="${width_base/2}" y="-${height_base/2 + height_wheel/2}" type="left" joint_type="fixed"/>
+    <xacro:wheel name ="front_right" x ="-${width_base/2}" y="${height_base/2 + height_wheel/2}" type="right" joint_type="continuous"/>
+    <xacro:wheel name ="front_left" x ="-${width_base/2}" y="-${height_base/2 + height_wheel/2}" type="left" joint_type="continuous"/>
+    <joint name="camera_joint" type="fixed">
+        <parent link="base_link"/>
+        <child link="camera_link"/>
+        <origin xyz="-${width_base/2 - 0.0125} 0 ${depth_base/2 + 0.0125}" rpy="0 0 3.14"/>
+        <axis xyz="0 0 0"/>
+    </joint>
+    <link name="camera_link">
         <visual>
             <geometry>
-                <box size="0.09 0.025 0.025" />
+                <box size="0.025 0.09 0.025" />
             </geometry>
             <material name="LightGrey">
@@ -93,11 +100,11 @@
         </inertial>
     </link>
-    <joint name="realsense_camera_joint" type="fixed">
-        <parent link="base_link"/>
-        <child link="realsense_camera_link"/>
-        <origin xyz="-0.2875 0 0.0625" rpy="0 0 -1.57"/>
-        <axis xyz="0 0 0"/>
-    </joint>
+  <!-- <joint name="imu_joint" type="fixed">
+    <parent link="base_link"/>
+    <child link="imu_link"/>
+    <origin xyz="-0.032 0 0.068" rpy="0 0 0"/>
+  </joint>
+  <link name="imu_link"/> -->
     <xacro:include filename="gazebo.xacro"/>
-    <xacro:include filename="testbot_d435i.xacro"/>
+    <!-- <xacro:include filename="testbot_d435i.xacro"/> -->
 </robot>

File: src/testbot_description/urdf/testbot_d435i.xacro (robot description, xacro)
@@ -9,8 +9,8 @@
        sideways (- right / + left)
        " -->
-  <xacro:sensor_d435i parent="realsense_camera_link" use_nominal_extrinsics="$(arg use_nominal_extrinsics)">
+  <xacro:sensor_d435i parent="testbot_camera_link" use_nominal_extrinsics="$(arg use_nominal_extrinsics)">
     <origin
       xyz="0 0 0.0125"
-      rpy="0.0 0.0 -1.57" />
+      rpy="0.0 0.0 0.0" />
   </xacro:sensor_d435i>
 </robot>
