Commit message: added 2d lidar

File: src/testbot_description/urdf/gazebo.xacro (robot description, xacro)
@@ -1,57 +1,60 @@
 <?xml version="1.0"?>
 <robot xmlns:xacro="http://www.ros.org/wiki/xacro">
-    <gazebo reference="base_link">
-        <material>Gazebo/Red</material>
-    </gazebo>
     <!-- Gazebo plugin for ROS Control -->
     <gazebo>
         <plugin name="gazebo_ros_control" filename="libgazebo_ros_control.so"/>
     </gazebo>
-    <!-- <xacro:macro name="wheel_trans" params="name mu1 mu2">
-        <transmission name="wheel_${name}_trans">
-            <type>transmission_interface/SimpleTransmission</type>
-            <actuator name="wheel_${name}_motor">
-                <mechanicalReduction>1</mechanicalReduction>
-            </actuator>
-            <joint name="wheel_${name}_joint">
-                <hardwareInterface>hardware_interface/VelocityJointInterface</hardwareInterface>
-            </joint>
-        </transmission>
-        <gazebo reference="wheel_${name}_link">
-            <mu1 value="${mu1}"/>
-            <mu2 value="${mu2}"/>
-            <kp value="10000000.0" />
-            <kd value="1.0" />
-            <material>Gazebo/DarkGrey</material>
-        </gazebo>
-    </xacro:macro> -->
-<gazebo reference="wheel_front_right_link">
-  <material>Gazebo/DarkGrey</material>
-  <mu1>0.5</mu1>
-  <mu2>0.5</mu2>
-  <selfCollide>true</selfCollide>
-</gazebo>
-<gazebo reference="wheel_front_left_link">
-  <material>Gazebo/DarkGrey</material>
-  <mu1>0.5</mu1>
-  <mu2>0.5</mu2>
-  <selfCollide>true</selfCollide>
-</gazebo>
-<gazebo reference="wheel_rear_right_link">
-  <material>Gazebo/DarkGrey</material>
-  <mu1>0.001</mu1>
-  <mu2>0.001</mu2>
-  <selfCollide>true</selfCollide>
-</gazebo>
-<gazebo reference="wheel_rear_left_link">
-  <material>Gazebo/DarkGrey</material>
-  <mu1>0.001</mu1>
-  <mu2>0.001</mu2>
-  <selfCollide>true</selfCollide>
-</gazebo>
-    <!-- <xacro:wheel_trans name ="rear_right" mu1 ="0.01" mu2 = "0.01"/>
-    <xacro:wheel_trans name ="rear_left" mu1 ="0.01" mu2 = "0.01"/> -->
-    <!-- <xacro:wheel_trans name ="front_right" mu1 ="200" mu2 = "100"/>
-    <xacro:wheel_trans name ="front_left" mu1 ="200" mu2 = "100"/> -->
+    <gazebo reference="base_link">
+        <material>Gazebo/Red</material>
+    </gazebo>
+    <gazebo reference="wheel_front_right_link">
+    <material>Gazebo/DarkGrey</material>
+    <mu1>0.5</mu1>
+    <mu2>0.5</mu2>
+    <selfCollide>true</selfCollide>
+    </gazebo>
+    <gazebo reference="wheel_front_left_link">
+    <material>Gazebo/DarkGrey</material>
+    <mu1>0.5</mu1>
+    <mu2>0.5</mu2>
+    <selfCollide>true</selfCollide>
+    </gazebo>
+    <gazebo reference="wheel_rear_right_link">
+    <material>Gazebo/DarkGrey</material>
+    <mu1>0.001</mu1>
+    <mu2>0.001</mu2>
+    <selfCollide>true</selfCollide>
+    </gazebo>
+    <gazebo reference="wheel_rear_left_link">
+    <material>Gazebo/DarkGrey</material>
+    <mu1>0.001</mu1>
+    <mu2>0.001</mu2>
+    <selfCollide>true</selfCollide>
+    </gazebo>
+    <gazebo reference="lidar_link">
+        <material>Gazebo/Grey</material>
+        <sensor name="lidar_link" type="ray">
+            <pose> 0 0 0 0 0 0 </pose>
+            <visualize>true</visualize>
+            <update_rate>10</update_rate>
+            <ray>
+                <scan>
+                    <horizontal>
+                        <samples>360</samples>
+                        <min_angle>-3.14</min_angle>
+                        <max_angle>3.14</max_angle>
+                    </horizontal>
+                </scan>
+                <range>
+                    <min>0.3</min>
+                    <max>12</max>
+                </range>
+            </ray>
+            <plugin name="laser_controller" filename="libgazebo_ros_laser.so">
+                <topicName>/scan</topicName>
+                <frame_name>lidar_link</frame_name>
+            </plugin>
+        </sensor>
+    </gazebo>
     <joint name="camera_optical_joint" type="fixed">
         <origin xyz="0 0 0" rpy="-1.571 0 -1.571" />

File: src/testbot_description/urdf/my_robot.urdf.xacro (robot description, xacro)
@@ -100,4 +100,56 @@
         </inertial>
     </link>
+    <joint name="lidar_base_joint" type="fixed">
+        <parent link="base_link"/>
+        <child link="lidar_base_link"/>
+        <origin xyz="0 0 ${depth_base/2 + 0.01}" rpy="0 0 0"/>
+        <axis xyz="0 0 0"/>
+    </joint>
+    <link name="lidar_base_link">
+        <visual>
+            <geometry>
+                <cylinder radius="0.02" length="0.02" />
+            </geometry>
+            <material name="LightGrey">
+                <color rgba="0.7 0.7 0.7 1.0"/>
+            </material>
+        </visual>
+        <collision>
+            <geometry>
+                <cylinder radius="0.04" length="0.05" />
+            </geometry>
+        </collision>
+        <inertial>
+            <mass value="0.05"/>
+            <origin xyz="0.0 0.0 0.0" rpy="0.0 0.0 0.0"/>
+            <inertia ixx="0.001" ixy="0.0" ixz="0.0" iyy="0.001" iyz="0.0" izz="0.001"/>
+        </inertial>
+    </link>
+    <joint name="lidar_joint" type="fixed">
+        <parent link="lidar_base_link"/>
+        <child link="lidar_link"/>
+        <origin xyz="0 0 0.025" rpy="0 0 0"/>
+        <axis xyz="0 0 0"/>
+    </joint>
+    <link name="lidar_link">
+        <visual>
+            <geometry>
+                <cylinder radius="0.04" length="0.03" />
+            </geometry>
+            <material name="LightGrey">
+                <color rgba="0.7 0.7 0.7 1.0"/>
+            </material>
+        </visual>
+        <collision>
+            <geometry>
+                <cylinder radius="0.04" length="0.05" />
+            </geometry>
+        </collision>
+        <inertial>
+            <mass value="0.05"/>
+            <origin xyz="0.0 0.0 0.0" rpy="0.0 0.0 0.0"/>
+            <inertia ixx="0.001" ixy="0.0" ixz="0.0" iyy="0.001" iyz="0.0" izz="0.001"/>
+        </inertial>
+    </link>
   <!-- <joint name="imu_joint" type="fixed">
     <parent link="base_link"/>
